File: SAM9260_QFP/sam9260_qfp/sam9260_qfp.kicad_sch (KiCad schematic)
At the start: 49 parts, among them J101 Conn_ARM_JTAG_SWD_10, SW101 SW_Push, SW102 SW_DIP_x01, U101 AT91SAM9260-QU, Y101 18MHz

Commit message: Completed component placing
Parts:
- added C135: 4.7u, Capacitor_SMD:C_0603_1608Metric, symbol Device:C_Small
- added FB101: 120R, Inductor_SMD:L_0603_1608Metric, symbol Device:FerriteBead_Small
- U101: footprint My_First_PCB:PQFP208_ATM -> SAM9260:PQFP208_ATM
Connections:
- net +3.3V: now also J101.1 (VTref), C135.1, FB101.1; no longer C112.1, C113.1, U101.160 (VDDANA)
- net GND: now also C135.2; no longer J101.1 (VTref)
- new net +3.3VA: C112.1, C113.1, FB101.2, U101.160 (VDDANA)
Other:
- moved on the sheet: C104, C105, C106, C107, C108, C109, C110, C112, C113, C114, C115, C116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

Commit message: updated layout
Parts:
- removed C132: 10u, Capacitor_SMD:C_0603_1608Metric, symbol Device:C_Small
- removed C135: 4.7u, Capacitor_SMD:C_0603_1608Metric, symbol Device:C_Small
- removed R103: 1k, Resistor_SMD:R_0402_1005Metric, symbol Device:R
- removed R108, R109: 100k, Resistor_SMD:R_0603_1608Metric, symbol Device:R_Small
- removed U101: AT91SAM9260-QU, SAM9260:PQFP208_ATM, symbol eec:AT91SAM9260-QU
- added C103: 10u, Capacitor_SMD:C_0603_1608Metric, symbol Device:C_Small
- added C111: 100n, Capacitor_SMD:C_0402_1005Metric, symbol Device:C_Small
- added H201, H202, H203, H204: MountingHole, MountingHole:MountingHole_3mm, symbol Mechanical:MountingHole
- added R103, R105: 100k, Resistor_SMD:R_0603_1608Metric, symbol Device:R_Small
- added R104: 1k, Resistor_SMD:R_0402_1005Metric, symbol Device:R
- added U101: AT91SAM9260B-QU, SAM9260:PQFP208_ATM, symbol SAM9260:AT91SAM9260B-QU
- C102, C121, C123, C131: value 100n -> 10u; footprint Capacitor_SMD:C_0402_1005Metric -> Capacitor_SMD:C_0603_1608Metric
- C104, C110, C114, C122: value 10u -> 100n; footprint Capacitor_SMD:C_0603_1608Metric -> Capacitor_SMD:C_0402_1005Metric
- C113: value 4.7u -> 100n; footprint Capacitor_SMD:C_0603_1608Metric -> Capacitor_SMD:C_0402_1005Metric
- C120, C125: value 100n -> 4.7u; footprint Capacitor_SMD:C_0402_1005Metric -> Capacitor_SMD:C_0603_1608Metric
- R101: value 1.5M -> 1k; footprint Resistor_SMD:R_0805_2012Metric -> Resistor_SMD:R_0402_1005Metric
- R102: value 1k -> 1.5M; footprint Resistor_SMD:R_0402_1005Metric -> Resistor_SMD:R_0805_2012Metric
- renumbered C103 to C132, C111 to C133, C133 to C134, C134 to C135, R104 to R108, R105 to R109
Connections:
- net +1V8: now also C102.2, C108.2, C114.2, C117.2, C121.2, C131.2, SW101.1, C111.2, U101.147 (VDDCORE), U101.148 (VDDPLL), U101.155 (VDDPLL), U101.174 (VDDCORE), U101.203 (VDDCORE), U101.38 (VDDCORE), U101.47 (VDDBU), U101.77 (VDDCORE); no longer C104.2, C123.2, C125.2, C126.2, C127.2, C128.2, C129.2, R101.1, SW101.2
- net +2V5: now also C123.1, C126.1, U101.169 (VDDIOP1); no longer C131.1
- net +3.3V: now also C104.2, C107.2, C110.2, C112.1, C113.2, C115.1, C120.1, C128.2, C129.2, C103.1, R103.1, R105.1, U101.114 (VDDIOM), U101.13 (VDDIOP0), U101.132 (VDDIOM), U101.187 (VDDIOP0), U101.199 (VDDIOP0), U101.24 (VDDIOP0), U101.32 (VDDIOP0), U101.5 (VDDIOP0), U101.52 (VDDIOP0), U101.65 (VDDIOM), U101.90 (VDDIOM); no longer C102.2, C107.1, C108.1, C110.1, C114.2, C115.2, C117.2, C120.2, C121.2
- net +3.3VA: now also C125.1, C127.1, U101.160 (VDDANA); no longer C112.1, C113.1
- net BMS: now also U101.40 (BMS)
- net GND: now also C107.1, C108.1, C110.1, C113.1, C115.2, C120.2, C123.2, C125.2, C126.2, C127.2, C131.1, R101.1, SW101.2, C103.2, C111.1, R104.1, U101.113 (GND), U101.133 (GND), U101.14 (GND), U101.146 (GND), U101.151 (GNDPLL), U101.153 (GNDPLL), U101.156 (GNDANA), U101.170 (GND), U101.173 (GND), U101.188 (GND), U101.200 (GND), U101.204 (GND), U101.25 (GND), U101.33 (GND), U101.39 (GND), U101.44 (GNDBU), U101.53 (GND), U101.6 (GND), U101.66 (GND), U101.78 (GND), U101.91 (GND); no longer C107.2, C108.2, C110.2, C113.2, C115.1, C120.1, C123.1, C125.1, C126.1, C127.1, C131.2, SW101.1
- net MDC: now also U101.205 (PA20)
- net MDIO: now also U101.206 (PA21)
- net PLLRCA: now also U101.154 (PLLRCA)
- net RX_D0: now also U101.195 (PA14)
- net RX_D1: now also U101.196 (PA15)
- net RX_D2: now also U101.2 (PA25)
- net RX_D3: now also U101.3 (PA26)
- net RX_DV: now also U101.198 (PA17)
- net SD_CLK: now also U101.189 (PA8)
- net SD_CMD: now also U101.186 (PA7)
- net SD_DAT0: now also U101.185 (PA6)
- net SD_DAT1: now also U101.190 (PA9)
- net SD_DAT2: now also U101.191 (PA10)
- net SD_DAT3: now also U101.192 (PA11)
- net TX_D0: now also U101.193 (PA12)
- net TX_D1: now also U101.194 (PA13)
- net TX_D2: now also U101.208 (PA23)
- net TX_D3: now also U101.1 (PA24)
- net TX_EN: now also U101.197 (PA16)
- net USB_CONN_HOST_D1_N: now also U101.54 (DDM)
- net USB_CONN_HOST_D1_P: now also U101.55 (DDP)
- net USB_CONN_HOST_D_N: now also U101.50 (HDMA)
- net USB_CONN_HOST_D_P: now also U101.51 (HDPA)
- net XIN: now also U101.149 (XIN)
- net XOUT: now also U101.150 (XOUT)
- net TMS_DBG: now reaches J101.2 (SWDIO/TMS)
- net TMS_DBG: now also R106.2, U101.31 (TMS)
- net NTRST_DBG: now reaches J101.10 (~{RESET})
- net NTRST_DBG: now also R103.2, U101.35 (NTRST); no longer R106.2
- net at R102.2: now also U101.49 (SHDN)
- net at R101.2: now also U101.42 (TST)
- net TCK_DBG: now reaches R107.2
- net TCK_DBG: now also J101.4 (SWDCLK/TCK), U101.34 (TCK); no longer J101.8 (NC/TDI)
- net TD0_DBG: now reaches J101.6 (SWO/TDO)
- net TD0_DBG: now also U101.29 (TDO)
- net JTAGSEL_DBG: now reaches SW102.1
- net JTAGSEL_DBG: now also U101.43 (JTAGSEL)
- new net: R104.2, U101.48 (WKUP)
- new net GTX_CLK_N: U101.202 (PA19)
- new net RX_CLK_N: U101.4 (PA27)
- new net TD1_DBG: J101.8 (NC/TDI), R105.2, U101.30 (TDI)
- no-connect marks 129 -> 128
Other:
- note added: "https://electronics.stackexchange.com/questions/37734/pull-down-resistors"
- moved on the sheet: C132, C133, C134, C135, JP101, R108, R109, Y101

Commit message: Completed routing, need to add logo
Changed lines of the file:
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@@
   (junction (at 25.4 158.75) (diameter 0) (color 0 0 0 0)
-  )
-  (junction (at 59.69 137.16) (diameter 0) (color 0 0 0 0)
   )
   (junction (at 132.08 161.29) (diameter 0) (color 0 0 0 0)
@@
     (stroke (width 0) (type default))
   )
-  (wire (pts (xy 59.69 137.16) (xy 64.77 137.16))
-    (stroke (width 0) (type default))
-  )
   (polyline (pts (xy 179.07 135.89) (xy 209.55 135.89))
     (stroke (width 0) (type default))
@@
     (stroke (width 0) (type default))
   )
-  (polyline (pts (xy 15.24 127) (xy 15.24 193.04))
+  (polyline (pts (xy 15.24 128.27) (xy 15.24 194.31))
     (stroke (width 0) (type default))
   )
@@
         )
       )
-    )
-  )
-  (symbol (lib_id "power:PWR_FLAG") (at 64.77 137.16 0) (unit 1)
-    (in_bom yes) (on_board yes) (dnp no)
-    (property "Reference" "#FLG0201" (at 64.77 135.255 0)
-      (effects (font (size 1.27 1.27)) hide)
-    )
-    (property "Value" "PWR_FLAG" (at 69.85 133.35 0)
-      (effects (font (size 1.27 1.27)))
-    )
-    (property "Footprint" "" (at 64.77 137.16 0)
-      (effects (font (size 1.27 1.27)) hide)
-    )
-    (property "Datasheet" "~" (at 64.77 137.16 0)
-      (effects (font (size 1.27 1.27)) hide)
-    )
-    (pin "1")
-    (instances
-      (project "sam9260_qfp"
-        (path "/e0cfbfe5-8f1c-42d1-90c4-1cf34dee8164"
-          (reference "#FLG0201") (unit 1)
-        )
-      )
